File: networking/rj45_breakout/rj45_breakout.kicad_sch (KiCad schematic)
At the start: 0 parts

Commit message: Fix: relinked footprints
Parts:
- added J1: RJ45_LED, symbol Connector:RJ45_LED
- added J2: RJ45_Amphenol_RJMG1BD3B8K1ANR, Connector_RJ:RJ45_Amphenol_RJMG1BD3B8K1ANR, symbol Connector:RJ45_Amphenol_RJMG1BD3B8K1ANR
Connections:
- new net RCT: J1.5, J2.R5 (RCT)
- new net RD+: J1.3, J2.R3 (RD+)
- new net RD-: J1.6, J2.R6 (RD-)
- new net TCT: J1.4, J2.R4 (TCT)
- new net TD+: J1.1, J2.R1 (TD+)
- new net TD-: J1.2, J2.R2 (TD-)
Changed lines of the file:
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@@
 (kicad_sch (version 20230409) (generator eeschema)
   (paper "A4")
-  (symbol_instances)
+  (wire (pts (xy 163.195 79.375) (xy 167.005 79.375))
+    (stroke (width 0) (type default))
+  )
+  (wire (pts (xy 161.925 100.33) (xy 165.735 100.33))
+    (stroke (width 0) (type default))
+  )
+  (wire (pts (xy 161.925 102.87) (xy 165.735 102.87))
+    (stroke (width 0) (type default))
+  )
+  (wire (pts (xy 161.925 97.79) (xy 165.735 97.79))
+    (stroke (width 0) (type default))
+  )
+  (wire (pts (xy 161.925 105.41) (xy 165.735 105.41))
+    (stroke (width 0) (type default))
+  )
+  (wire (pts (xy 161.925 95.25) (xy 165.735 95.25))
+    (stroke (width 0) (type default))
+  )
+  (wire (pts (xy 163.195 76.835) (xy 167.005 76.835))
+    (stroke (width 0) (type default))
+  )
+  (wire (pts (xy 163.195 71.755) (xy 167.005 71.755))
+    (stroke (width 0) (type default))
+  )
+  (wire (pts (xy 163.195 69.215) (xy 167.005 69.215))
+    (stroke (width 0) (type default))
+  )
+  (wire (pts (xy 163.195 74.295) (xy 167.005 74.295))
+    (stroke (width 0) (type default))
+  )
+  (wire (pts (xy 163.195 81.915) (xy 167.005 81.915))
+    (stroke (width 0) (type default))
+  )
+  (wire (pts (xy 161.925 107.95) (xy 165.735 107.95))
+    (stroke (width 0) (type default))
+  )
+  (label "RD-" (at 161.925 107.95 0) (fields_autoplaced)
+    (effects (font (size 1.27 1.27)) (justify left bottom))
+  )
+  (label "RCT" (at 161.925 105.41 0) (fields_autoplaced)
+    (effects (font (size 1.27 1.27)) (justify left bottom))
+  )
+  (label "RD-" (at 163.195 81.915 0) (fields_autoplaced)
+    (effects (font (size 1.27 1.27)) (justify left bottom))
+  )
+  (label "TCT" (at 161.925 97.79 0) (fields_autoplaced)
+    (effects (font (size 1.27 1.27)) (justify left bottom))
+  )
+  (label "RD+" (at 161.925 102.87 0) (fields_autoplaced)
+    (effects (font (size 1.27 1.27)) (justify left bottom))
+  )
+  (label "TD+" (at 163.195 69.215 0) (fields_autoplaced)
+    (effects (font (size 1.27 1.27)) (justify left bottom))
+  )
+  (label "TD-" (at 161.925 100.33 0) (fields_autoplaced)
+    (effects (font (size 1.27 1.27)) (justify left bottom))
+  )
+  (label "TD-" (at 163.195 71.755 0) (fields_autoplaced)
+    (effects (font (size 1.27 1.27)) (justify left bottom))
+  )
+  (label "TD+" (at 161.925 95.25 0) (fields_autoplaced)
+    (effects (font (size 1.27 1.27)) (justify left bottom))
+  )
+  (label "RD+" (at 163.195 74.295 0) (fields_autoplaced)
+    (effects (font (size 1.27 1.27)) (justify left bottom))
+  )
+  (label "TCT" (at 163.195 76.835 0) (fields_autoplaced)
+    (effects (font (size 1.27 1.27)) (justify left bottom))
+  )
+  (label "RCT" (at 163.195 79.375 0) (fields_autoplaced)
+    (effects (font (size 1.27 1.27)) (justify left bottom))
+  )
+  (symbol (lib_id "Connector:RJ45_LED") (at 177.165 76.835 180) (unit 1)
+    (in_bom yes) (on_board yes) (dnp no) (fields_autoplaced)
+    (property "Reference" "J1" (at 177.165 62.23 0)
+      (effects (font (size 1.27 1.27)))
+    )
+    (property "Value" "RJ45_LED" (at 177.165 64.77 0)
+      (effects (font (size 1.27 1.27)))
+    )
+    (property "Footprint" "" (at 177.165 77.47 90)
+      (effects (font (size 1.27 1.27)) hide)
+    )
+    (property "Datasheet" "~" (at 177.165 77.47 90)
+      (effects (font (size 1.27 1.27)) hide)
+    )
+    (pin "1")
+    (pin "10")
+    (pin "11")
+    (pin "12")
+    (pin "2")
+    (pin "3")
+    (pin "4")
+    (pin "5")
+    (pin "6")
+    (pin "7")
+    (pin "8")
+    (pin "9")
+    (instances
+      (project "rj45_breakout"
+        (path "/b89c3d15-0b9e-4adf-8b6e-6cf4bb84cb6a"
+          (reference "J1") (unit 1)
+        )
+      )
+    )
+  )
+  (symbol (lib_id "Connector:RJ45_Amphenol_RJMG1BD3B8K1ANR") (at 188.595 107.95 0) (unit 1)
+    (in_bom yes) (on_board yes) (dnp no) (fields_autoplaced)
+    (property "Reference" "J2" (at 188.595 90.17 0)
+      (effects (font (size 1.27 1.27)))
+    )
+    (property "Value" "RJ45_Amphenol_RJMG1BD3B8K1ANR" (at 188.595 92.71 0)
+      (effects (font (size 1.27 1.27)))
+    )
+    (property "Footprint" "Connector_RJ:RJ45_Amphenol_RJMG1BD3B8K1ANR" (at 188.595 90.17 0)
+      (effects (font (size 1.27 1.27)) hide)
+    )
+    (property "Datasheet" "https://www.amphenolcanada.com/ProductSearch/Drawings/AC/RJMG1BD3B8K1ANR.PDF" (at 188.595 87.63 0)
+      (effects (font (size 1.27 1.27)) hide)
+    )
+    (pin "13")
+    (pin "L1")
+    (pin "L2")
+    (pin "L3")
+    (pin "L4")
+    (pin "R1")
+    (pin "R2")
+    (pin "R3")
+    (pin "R4")
+    (pin "R5")
+    (pin "R6")
+    (pin "R7")
+    (pin "R8")
+    (instances
+      (project "rj45_breakout"
+        (path "/b89c3d15-0b9e-4adf-8b6e-6cf4bb84cb6a"
+          (reference "J2") (unit 1)
+        )
+      )
+    )
+  )
+  (sheet_instances
+    (path "/" (page "1"))
+  )
 )
