File: carrier/carrier.kicad_pcb (KiCad board)
At the start: 2 copper layers, 0 parts

Commit message: Fix: fixed 3D models for carrier board
Parts:
- added BZ1: Buzzer, Buzzer_Beeper:Buzzer_TDK_PS1240P02BT_D12.2mm_H6.5mm, F.Cu at (101.7, 110.8)
- added C1: 100n, Capacitor_SMD:C_0402_1005Metric, F.Cu at (107.5, 61.1)
- added C10: 100n, Capacitor_SMD:C_0402_1005Metric, F.Cu at (147.3, 54.7)
- added C11: 100n, Capacitor_SMD:C_0402_1005Metric, F.Cu at (147.3, 56.7)
- added C12: 100uF, Capacitor_Tantalum_SMD:CP_EIA-7343-31_Kemet-D, F.Cu at (145.0, 67.6)
- added C13: 100n, Capacitor_SMD:C_0402_1005Metric, F.Cu at (147.3, 58.6)
- added C14: 10u, Capacitor_SMD:C_0805_2012Metric, F.Cu at (123.2, 56.4)
- added C15: 100n, Capacitor_SMD:C_0402_1005Metric, F.Cu at (147.3, 60.6)
- added C16: 10u, Capacitor_SMD:C_0805_2012Metric, F.Cu at (123.2, 59.4)
- added C17: 10u, Capacitor_SMD:C_0805_2012Metric, F.Cu at (123.2, 62.4)
- added C18: 10u, Capacitor_SMD:C_0805_2012Metric, F.Cu at (123.2, 65.4)
- added C19: 100n, Capacitor_SMD:C_0402_1005Metric, F.Cu at (139.5, 140.1)
- added C2: 100n, Capacitor_SMD:C_0402_1005Metric, F.Cu at (107.5, 63.1)
- added C20: 10uF, Capacitor_SMD:C_0603_1608Metric, F.Cu at (103.7, 118.9)
- added C21: 0.1uF, Capacitor_SMD:C_0603_1608Metric, F.Cu at (103.7, 121.5)
- added C22: 10uF, Capacitor_SMD:C_0603_1608Metric, F.Cu at (103.7, 124.0)
- added C23: 10uF, Capacitor_SMD:C_0603_1608Metric, F.Cu at (103.7, 126.5)
- added C24: 100nF, Capacitor_SMD:C_0603_1608Metric, F.Cu at (103.7, 129.0)
- added C25: 10uF, Capacitor_SMD:C_0603_1608Metric, F.Cu at (107.7, 118.9)
- added C26: 100nF, Capacitor_SMD:C_0603_1608Metric, F.Cu at (107.7, 121.5)
- added C27: 10uF, Capacitor_SMD:C_0603_1608Metric, F.Cu at (107.7, 124.0)
- added C28: 1uF, Capacitor_SMD:C_0603_1608Metric, F.Cu at (107.7, 126.5)
- added C29: 100nF, Capacitor_SMD:C_0603_1608Metric, F.Cu at (107.7, 129.0)
- added C3: 27pF, Capacitor_SMD:C_0402_1005Metric, F.Cu at (147.3, 46.8)
- added C30: 0.1uF, Capacitor_SMD:C_0603_1608Metric, F.Cu at (158.8, 105.2)
- added C31: 0.1uF, Capacitor_SMD:C_0603_1608Metric, F.Cu at (158.8, 107.7)
- added C32: 0.1uF, Capacitor_SMD:C_0603_1608Metric, F.Cu at (158.8, 110.2)
- added C33: 0.1uF, Capacitor_SMD:C_0603_1608Metric, F.Cu at (158.8, 112.7)
- added C34: 0.1uF, Capacitor_SMD:C_0603_1608Metric, F.Cu at (158.8, 115.2)
- added C35: 0.1uF, Capacitor_SMD:C_0603_1608Metric, F.Cu at (158.8, 117.7)
- added C4: 10u, Capacitor_SMD:C_0805_2012Metric, F.Cu at (123.2, 47.3)
- added C5: 10u, Capacitor_SMD:C_0805_2012Metric, F.Cu at (123.2, 50.3)
- added C6: 10u, Capacitor_SMD:C_0805_2012Metric, F.Cu at (123.2, 53.3)
- added C7: 27pF, Capacitor_SMD:C_0402_1005Metric, F.Cu at (147.3, 48.8)
- added C8: 100n, Capacitor_SMD:C_0402_1005Metric, F.Cu at (147.3, 50.7)
- added C9: 100n, Capacitor_SMD:C_0402_1005Metric, F.Cu at (147.3, 52.7)
- added D1: LED Green, LED_SMD:LED_0603_1608Metric, F.Cu at (136.0, 140.4)
- added D2: LED Red, LED_SMD:LED_0603_1608Metric, F.Cu at (136.0, 143.0)
- added D3: 1N4148, Diode_SMD:D_0603_1608Metric, F.Cu at (99.1, 144.9)
- added D4: WS2812B, LED_SMD:LED_WS2812B_PLCC4_5.0x5.0mm_P3.2mm, F.Cu at (152.6, 107.2)
- added D5: WS2812B, LED_SMD:LED_WS2812B_PLCC4_5.0x5.0mm_P3.2mm, F.Cu at (152.6, 113.9)
- added D6: WS2812B, LED_SMD:LED_WS2812B_PLCC4_5.0x5.0mm_P3.2mm, F.Cu at (152.6, 120.5)
- added D7: WS2812B, LED_SMD:LED_WS2812B_PLCC4_5.0x5.0mm_P3.2mm, F.Cu at (152.6, 127.1)
- added D8: WS2812B, LED_SMD:LED_WS2812B_PLCC4_5.0x5.0mm_P3.2mm, F.Cu at (152.6, 133.7)
- added D9: WS2812B, LED_SMD:LED_WS2812B_PLCC4_5.0x5.0mm_P3.2mm, F.Cu at (152.6, 140.3)
- added H1: MountingHole, MountingHole:MountingHole_2.7mm_M2.5, F.Cu at (63.5, 107.4)
- added H2: MountingHole, MountingHole:MountingHole_2.7mm_M2.5, F.Cu at (63.5, 114.4)
- added H3: MountingHole, MountingHole:MountingHole_2.7mm_M2.5, F.Cu at (70.5, 107.4)
- added H4: MountingHole, MountingHole:MountingHole_2.7mm_M2.5, F.Cu at (70.5, 114.4)
- added H5: MountingHole, MountingHole:MountingHole_2.7mm_M2.5, F.Cu at (77.4, 107.4)
- added H6: MountingHole, MountingHole:MountingHole_2.7mm_M2.5, F.Cu at (77.4, 114.4)
- added H7: MountingHole, MountingHole:MountingHole_2.7mm_M2.5, F.Cu at (84.4, 107.4)
- added H8: MountingHole, MountingHole:MountingHole_2.7mm_M2.5, F.Cu at (84.4, 114.4)
- added J1: 690-019-298-412, CM4IO:EDAC 690-019-298-412, F.Cu at (110.0, 49.0)
- added J10: Conn_01x04, Connector_PinHeader_2.54mm:PinHeader_1x04_P2.54mm_Vertical, F.Cu at (113.4, 106.3)
- added J11: Conn_01x08, Connector_PinHeader_2.54mm:PinHeader_1x08_P2.54mm_Vertical, F.Cu at (99.4, 120.0)
- added J2: USB_C_Receptacle_USB2.0, Connector_USB:USB_C_Receptacle_HRO_TYPE-C-31-M-12, F.Cu at (131.3, 76.7)
- added J3: Conn_02x05_Odd_Even, Connector_PinHeader_2.54mm:PinHeader_2x05_P2.54mm_Vertical, F.Cu at (151.1, 48.1)
- added J4: 690-008-221-904, CM4IO:MOLEX_USB_67298-4090, F.Cu at (134.2, 53.7)
- added J5: Conn_02x07_Odd_Even, Connector_PinHeader_2.54mm:PinHeader_2x07_P2.54mm_Vertical, F.Cu at (129.1, 129.3)
- added J6: Conn_01x03, Connector_PinHeader_2.54mm:PinHeader_1x03_P2.54mm_Vertical, F.Cu at (129.1, 149.2)
- added J7: THD-20-R, Connector_PinHeader_2.54mm:PinHeader_2x20_P2.54mm_Vertical, F.Cu at (121.9, 106.3)
- added J9: Conn_02x16_Top_Bottom, Connector_PinHeader_2.54mm:PinHeader_2x16_P2.54mm_Vertical, F.Cu at (92.2, 106.3)
- added JP1: TO_GND, Jumper:SolderJumper-2_P1.3mm_Open_RoundedPad1.0x1.5mm, F.Cu at (99.2, 141.9)
- added Module1: ComputeModule4, CM4IO:Raspberry-Pi-4-Compute-Module, F.Cu at (64.1, 97.9)
- added R1: 36K 1%, Resistor_SMD:R_0402_1005Metric, F.Cu at (144.5, 46.8)
- added R10: 5.1k, Resistor_SMD:R_0603_1608Metric, F.Cu at (152.0, 68.5)
- added R11: 1k, Resistor_SMD:R_0402_1005Metric, F.Cu at (139.5, 127.9)
- added R12: 1k, Resistor_SMD:R_0402_1005Metric, F.Cu at (139.5, 129.9)
- added R13: 470R, Resistor_SMD:R_0402_1005Metric, F.Cu at (139.5, 131.9)
- added R14: 470R, Resistor_SMD:R_0402_1005Metric, F.Cu at (139.5, 133.9)
- added R15: 10k, Resistor_SMD:R_0603_1608Metric, F.Cu at (111.7, 118.9)
- added R16: 10k, Resistor_SMD:R_0603_1608Metric, F.Cu at (111.7, 121.5)
- added R17: 10k, Resistor_SMD:R_0603_1608Metric, F.Cu at (111.7, 124.0)
- added R18: 10k, Resistor_SMD:R_0603_1608Metric, F.Cu at (62.0, 119.1)
- added R19: 10k, Resistor_SMD:R_0603_1608Metric, F.Cu at (62.0, 121.6)
- added R2: 36K 1%, Resistor_SMD:R_0402_1005Metric, F.Cu at (144.5, 48.8)
- added R20: 470, Resistor_SMD:R_0603_1608Metric, F.Cu at (158.8, 120.3)
- added R3: 36K 1%, Resistor_SMD:R_0402_1005Metric, F.Cu at (144.5, 50.8)
- added R4: 12K 1%, Resistor_SMD:R_0402_1005Metric, F.Cu at (144.5, 52.8)
- added R5: 36K 1%, Resistor_SMD:R_0402_1005Metric, F.Cu at (144.5, 54.8)
- added R6: 15K 1%, Resistor_SMD:R_0402_1005Metric, F.Cu at (144.5, 56.8)
- added R7: 2.2K 1%, Resistor_SMD:R_0402_1005Metric, F.Cu at (144.5, 58.8)
- added R8: 2.2K 1%, Resistor_SMD:R_0402_1005Metric, F.Cu at (144.5, 60.7)
- added R9: 5.1k, Resistor_SMD:R_0603_1608Metric, F.Cu at (152.0, 66.0)
- added TP1: TestPoint, TestPoint:TestPoint_Pad_2.0x2.0mm, F.Cu at (136.0, 129.0)
- added TP2: TestPoint, TestPoint:TestPoint_Pad_2.0x2.0mm, F.Cu at (136.0, 133.0)
- added TP3: TestPoint, TestPoint:TestPoint_Pad_2.0x2.0mm, F.Cu at (103.7, 132.3)
- added TP4: TestPoint, TestPoint:TestPoint_Pad_2.0x2.0mm, F.Cu at (103.7, 136.3)
- added TP5: TestPoint, TestPoint:TestPoint_Pad_2.0x2.0mm, F.Cu at (103.7, 140.4)
- added TP6: TestPoint, TestPoint:TestPoint_Pad_2.0x2.0mm, F.Cu at (103.7, 144.4)
- added U1: RT9742SNGV, Package_TO_SOT_SMD:SOT-23, F.Cu at (103.6, 62.4)
- added U10: MagJack-A70-112-331N126, CM4IO:TRJG0926HENL, F.Cu at (136.6, 115.2)
- added U11: BME680, Package_LGA:Bosch_LGA-8_3x3mm_P0.8mm_ClockwisePinNumbering, F.Cu at (114.1, 143.8)
- added U12: PCA9685PW, Package_SO:TSSOP-28_4.4x9.7mm_P0.65mm, F.Cu at (110.1, 135.9)
- added U13: BMI088, BMI088:PQFN50P450X300X100-16N, F.Cu at (108.8, 144.3)
- added U14: MMC5603NJ, MMC5603NJ:XDCR_MMC5603NJ, F.Cu at (115.7, 119.6)
- added U15: SN74LV1T34DBV, Package_TO_SOT_SMD:SOT-23-5, F.Cu at (159.3, 123.7)
- added U2: AP22653W6, Package_TO_SOT_SMD:SOT-23-6, F.Cu at (150.9, 77.5)
- added U3: USB2514B-I/M2, Package_DFN_QFN:QFN-36-1EP_6x6mm_P0.5mm_EP3.7x3.7mm, F.Cu at (144.2, 74.7)
- added U4: FSUSB42MUX, Package_SO:MSOP-10_3x3mm_P0.5mm, F.Cu at (152.0, 72.9)
- added U5: TPD4EUSB30, Package_SON:USON-10_2.5x1.0mm_P0.5mm, F.Cu at (138.5, 73.0)
- added U6: 74LVC1G07SE-7, Package_TO_SOT_SMD:SOT-353_SC-70-5, F.Cu at (143.1, 128.9)
- added U7: TPD4EUSB30, Package_SON:USON-10_2.5x1.0mm_P0.5mm, F.Cu at (135.4, 137.1)
- added U8: TPD4EUSB30, Package_SON:USON-10_2.5x1.0mm_P0.5mm, F.Cu at (138.3, 137.1)
- added U9: 74LVC1G07SE-7, Package_TO_SOT_SMD:SOT-353_SC-70-5, F.Cu at (143.1, 132.7)
- added Y1: 24MHz, Crystal:Crystal_SMD_HC49-SD, F.Cu at (132.7, 67.8)

Commit message: Feat: begun work on carrier pcb and imported NGFF m.2 library
Parts:
- removed J11: Conn_01x08, Connector_PinHeader_2.54mm:PinHeader_1x08_P2.54mm_Vertical
- added D19: 1N4148, Diode_SMD:D_0603_1608Metric, F.Cu at (-25.5, 70.1)
- added D20: 1N4148, Diode_SMD:D_0603_1608Metric, F.Cu at (-25.5, 72.6)
- added D21: 1N4148, Diode_SMD:D_0603_1608Metric, F.Cu at (-25.5, 75.2)
- added D22: 1N4148, Diode_SMD:D_0603_1608Metric, F.Cu at (-25.5, 77.8)
- added D23: 1N4148, Diode_SMD:D_0603_1608Metric, F.Cu at (-25.5, 80.4)
- added D24: 1N4148, Diode_SMD:D_0603_1608Metric, F.Cu at (-25.5, 83.0)
- added D25: 1N4148, Diode_SMD:D_0603_1608Metric, F.Cu at (-25.5, 85.6)
- added D26: 1N4148, Diode_SMD:D_0603_1608Metric, F.Cu at (-25.5, 88.2)
- added D27: 1N4148, Diode_SMD:D_0603_1608Metric, F.Cu at (-25.5, 90.8)
- added J12: Conn_02x40_Odd_Even, M.2:NGFF_A, F.Cu at (11.0, 4.03)
- added J8: Conn_02x16_Top_Bottom, Connector_PinHeader_2.54mm:PinHeader_2x16_P2.54mm_Vertical, F.Cu at (117.4, 170.0)
- added JP2: Jumper, Jumper:SolderJumper-2_P1.3mm_Bridged_Pad1.0x1.5mm, F.Cu at (2.71, 70.5)
- added JP3: Jumper, Jumper:SolderJumper-2_P1.3mm_Bridged_Pad1.0x1.5mm, F.Cu at (2.71, 74.1)
- added JP4: Jumper, Jumper:SolderJumper-2_P1.3mm_Bridged_Pad1.0x1.5mm, F.Cu at (2.71, 77.6)
- added JP5: Jumper, Jumper:SolderJumper-2_P1.3mm_Bridged_Pad1.0x1.5mm, F.Cu at (2.71, 81.2)
- added JP6: Jumper, Jumper:SolderJumper-2_P1.3mm_Bridged_Pad1.0x1.5mm, F.Cu at (2.71, 84.7)
- added JP7: Jumper, Jumper:SolderJumper-2_P1.3mm_Bridged_Pad1.0x1.5mm, F.Cu at (2.71, 88.3)
- added SW10: KEYSW, Connector_JST:JST_GH_BM02B-GHS-TBT_1x02-1MP_P1.25mm_Vertical, F.Cu at (-19.5, 72.6)
- added SW11: KEYSW, Connector_JST:JST_GH_BM02B-GHS-TBT_1x02-1MP_P1.25mm_Vertical, F.Cu at (-19.5, 80.2)
- added SW12: KEYSW, Connector_JST:JST_GH_BM02B-GHS-TBT_1x02-1MP_P1.25mm_Vertical, F.Cu at (-19.5, 87.9)
- added SW13: KEYSW, Connector_JST:JST_GH_BM02B-GHS-TBT_1x02-1MP_P1.25mm_Vertical, F.Cu at (-11.5, 72.6)
- added SW14: KEYSW, Connector_JST:JST_GH_BM02B-GHS-TBT_1x02-1MP_P1.25mm_Vertical, F.Cu at (-11.5, 80.2)
- added SW15: KEYSW, Connector_JST:JST_GH_BM02B-GHS-TBT_1x02-1MP_P1.25mm_Vertical, F.Cu at (-11.5, 87.9)
- added SW16: KEYSW, Connector_JST:JST_GH_BM02B-GHS-TBT_1x02-1MP_P1.25mm_Vertical, F.Cu at (-3.46, 72.6)
- added SW17: KEYSW, Connector_JST:JST_GH_BM02B-GHS-TBT_1x02-1MP_P1.25mm_Vertical, F.Cu at (-3.46, 80.2)
- added SW18: KEYSW, Connector_JST:JST_GH_BM02B-GHS-TBT_1x02-1MP_P1.25mm_Vertical, F.Cu at (-3.46, 87.9)
- added TP23: ~, TestPoint:TestPoint_Pad_D1.5mm, F.Cu at (12.0, 33.7)
- added TP24: ~, TestPoint:TestPoint_Pad_D1.5mm, F.Cu at (15.6, 12.4)
- added TP25: ~, TestPoint:TestPoint_Pad_D1.5mm, F.Cu at (15.6, 16.0)
- added TP26: ~, TestPoint:TestPoint_Pad_D1.5mm, F.Cu at (15.6, 19.5)
- added TP27: ~, TestPoint:TestPoint_Pad_D1.5mm, F.Cu at (15.6, 23.1)
- added TP28: ~, TestPoint:TestPoint_Pad_D1.5mm, F.Cu at (15.6, 26.6)
- added TP29: ~, TestPoint:TestPoint_Pad_D1.5mm, F.Cu at (15.6, 30.2)
- added TP30: ~, TestPoint:TestPoint_Pad_D1.5mm, F.Cu at (15.6, 33.7)
- added TP31: ~, TestPoint:TestPoint_Pad_D1.5mm, F.Cu at (19.1, 12.4)
- added TP32: ~, TestPoint:TestPoint_Pad_D1.5mm, F.Cu at (19.1, 16.0)
- added TP33: ~, TestPoint:TestPoint_Pad_D1.5mm, F.Cu at (19.1, 19.5)
- added TP34: ~, TestPoint:TestPoint_Pad_D1.5mm, F.Cu at (19.1, 23.1)
- added TP35: ~, TestPoint:TestPoint_Pad_D1.5mm, F.Cu at (45.8, 88.1)
- added TP36: ~, TestPoint:TestPoint_Pad_D1.5mm, F.Cu at (45.8, 91.7)
- C21: value 0.1uF -> 100nF
- C23: value 10uF -> 0.1uF
- C24, C26: value 100nF -> 10uF
- C25: value 10uF -> 100nF
- J10: value Conn_01x04 -> Conn_01x08; footprint Connector_PinHeader_2.54mm:PinHeader_1x04_P2.54mm_Vertical -> Connector_PinHeader_2.54mm:PinHeader_1x08_P2.54mm_Vertical
- J3: value Conn_02x05_Odd_Even -> Conn_02x04; footprint Connector_PinHeader_2.54mm:PinHeader_2x05_P2.54mm_Vertical -> Connector_PinHeader_2.54mm:PinHeader_2x04_P2.54mm_Vertical
- J9: value Conn_02x16_Top_Bottom -> Conn_01x04; footprint Connector_PinHeader_2.54mm:PinHeader_2x16_P2.54mm_Vertical -> Connector_PinHeader_2.54mm:PinHeader_1x04_P2.54mm_Vertical
- R1, R2: value 36K 1% -> 10k; footprint Resistor_SMD:R_0402_1005Metric -> Resistor_SMD:R_0603_1608Metric
- R10, R9: value 5.1k -> 2.2K 1%; footprint Resistor_SMD:R_0603_1608Metric -> Resistor_SMD:R_0402_1005Metric
- R11, R12: value 1k -> 5.1k; footprint Resistor_SMD:R_0402_1005Metric -> Resistor_SMD:R_0603_1608Metric
- R13, R14: value 470R -> 1k
- R15, R16: value 10k -> 470R; footprint Resistor_SMD:R_0603_1608Metric -> Resistor_SMD:R_0402_1005Metric
- R4: value 12K 1% -> 36K 1%
- R6: value 15K 1% -> 12K 1%
- R7: value 2.2K 1% -> 36K 1%
- R8: value 2.2K 1% -> 15K 1%
- TP3, TP4, TP5, TP6: value TestPoint -> ~; footprint TestPoint:TestPoint_Pad_2.0x2.0mm -> TestPoint:TestPoint_Pad_D1.5mm
- U12: value PCA9685PW -> BMI088; footprint Package_SO:TSSOP-28_4.4x9.7mm_P0.65mm -> BMI088:PQFN50P450X300X100-16N
- U13: value BMI088 -> MMC5603NJ; footprint BMI088:PQFN50P450X300X100-16N -> MMC5603NJ:XDCR_MMC5603NJ
- U14: value MMC5603NJ -> PCA9685PW; footprint MMC5603NJ:XDCR_MMC5603NJ -> Package_SO:TSSOP-28_4.4x9.7mm_P0.65mm
- moved R9 211.1 mm to (-56.3, 100.6)
- moved R10 211.1 mm to (-56.3, 102.6)
- moved C10 205.1 mm to (-53.4, 96.5)
- moved C11 205.1 mm to (-53.4, 98.5)
- moved C13 205.1 mm to (-53.4, 100.4)
- moved C15 205.1 mm to (-53.4, 102.4)
- moved C3 205.1 mm to (-53.4, 88.6)
- moved C7 205.1 mm to (-53.4, 90.6)
- moved C8 205.1 mm to (-53.4, 92.6)
- moved C9 205.1 mm to (-53.4, 94.5)
- moved R3 204.3 mm to (-56.3, 88.6)
- moved R4 204.3 mm to (-56.3, 90.6)
- moved R5 204.3 mm to (-56.3, 92.6)
- moved R6 204.3 mm to (-56.3, 94.6)
- moved R7 204.3 mm to (-56.3, 96.6)
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Connections:
- C22 pad 1: GND -> /+3.3v
- C22 pad 2: /+3.3v -> GND
- C26 pad 1: /+3.3v -> GND
- C26 pad 2: GND -> /+3.3v
- D5 pad 3: unconnected-(D5-VSS-Pad3) -> GND
- D6 pad 3: unconnected-(D6-VSS-Pad3) -> GND
- D7 pad 3: unconnected-(D7-VSS-Pad3) -> GND
- D8 pad 3: unconnected-(D8-VSS-Pad3) -> GND
- D9 pad 3: unconnected-(D9-VSS-Pad3) -> GND
- J10 pad 1: /+3.3v -> /CM4_GPIO ( Ethernet, GPIO, SDCARD)/SDA0
- J10 pad 3: /CM4_GPIO ( Ethernet, GPIO, SDCARD)/SDA0 -> unconnected-(J10-Pin_3-Pad3)
- J10 pad 4: GND -> unconnected-(J10-Pin_4-Pad4)
- J3 pad 2: /USB2-HUB/VBUS -> /USB2-HUB/HD3_N
- J3 pad 3: /USB2-HUB/HD3_N -> /USB2-HUB/HD3_P
- J3 pad 4: /USB2-HUB/HD4_N -> GND
- J3 pad 5: /USB2-HUB/HD3_P -> /USB2-HUB/VBUS
- J3 pad 6: /USB2-HUB/HD4_P -> /USB2-HUB/HD4_N
- J3 pad 7: GND -> /USB2-HUB/HD4_P
- J9 pad 1: /Sensors/LED0 -> /+3.3v
- J9 pad 2: Net-(J9-Pin_2) -> /CM4_GPIO ( Ethernet, GPIO, SDCARD)/SCL0
- J9 pad 3: Net-(J9-Pin_3) -> /CM4_GPIO ( Ethernet, GPIO, SDCARD)/SDA0
- J9 pad 4: Net-(J9-Pin_4) -> GND
- R1 pad 1: Net-(U3-SCL/SMBCLK/CFG_SEL0) -> /+3.3v
- R1 pad 2: GND -> /CM4_GPIO ( Ethernet, GPIO, SDCARD)/SCL0
- R10 pad 1: /USB2-HUB/CC2 -> /USB2-HUB/VBUS
- R10 pad 2: GND -> /CM4_HighSpeed/USBOTG_ID
- R11 pad 1: Net-(D1-K) -> /USB2-HUB/CC1
- R11 pad 2: Net-(Module1A-PI_nLED_Activity) -> GND
- R12 pad 1: Net-(D2-K) -> /USB2-HUB/CC2
- R12 pad 2: Net-(R12-Pad2) -> GND
- R13 pad 1: Net-(U10-LEDG_K) -> Net-(D1-K)
- R13 pad 2: /CM4_GPIO ( Ethernet, GPIO, SDCARD)/ETH_LEDG -> Net-(Module1A-PI_nLED_Activity)
- R14 pad 1: Net-(U10-LEDY_K) -> Net-(D2-K)
- R14 pad 2: /CM4_GPIO ( Ethernet, GPIO, SDCARD)/ETH_LEDY -> Net-(R14-Pad2)
- R15 pad 1: /+3.3v -> Net-(U10-LEDG_K)
- R15 pad 2: Net-(JP1-B) -> /CM4_GPIO ( Ethernet, GPIO, SDCARD)/ETH_LEDG
- R16 pad 1: +3.3V -> Net-(U10-LEDY_K)
- R16 pad 2: Net-(D3-A) -> /CM4_GPIO ( Ethernet, GPIO, SDCARD)/ETH_LEDY
- R17 pad 1: Net-(U12-~{OE}) -> /+3.3v
- R17 pad 2: GND -> Net-(JP1-B)
- R18 pad 1: /+3.3v -> +3.3V
- R18 pad 2: /CM4_GPIO ( Ethernet, GPIO, SDCARD)/SCL0 -> Net-(D3-A)
- R19 pad 1: /CM4_GPIO ( Ethernet, GPIO, SDCARD)/SDA0 -> Net-(U14-~{OE})
- R19 pad 2: /+3.3v -> GND
- R2 pad 1: Net-(U3-SDA/SMBDATA/NON_REM1) -> /CM4_GPIO ( Ethernet, GPIO, SDCARD)/SDA0
- R2 pad 2: GND -> /+3.3v
- R3 pad 1: Net-(U3-SUSP_IND/LOCAL_PWR/NON_REM0) -> Net-(U3-SCL/SMBCLK/CFG_SEL0)
- R4 pad 1: GND -> Net-(U3-SDA/SMBDATA/NON_REM1)
- R4 pad 2: Net-(U3-RBIAS) -> GND
- R5 pad 1: Net-(U3-HS_IND/CFG_SEL1) -> Net-(U3-SUSP_IND/LOCAL_PWR/NON_REM0)
- R6 pad 1: Net-(U2-ILIM) -> GND
- R6 pad 2: GND -> Net-(U3-RBIAS)
- R7 pad 1: /CM4_HighSpeed/USBOTG_ID -> Net-(U3-HS_IND/CFG_SEL1)
- R8 pad 1: /USB2-HUB/VBUS -> Net-(U2-ILIM)
- R8 pad 2: /CM4_HighSpeed/USBOTG_ID -> GND
- R9 pad 1: /USB2-HUB/CC1 -> /CM4_HighSpeed/USBOTG_ID
- TP3 pad 1: Net-(U13-INT1) -> Net-(U12-INT1)
- TP4 pad 1: Net-(U13-INT2) -> Net-(U12-INT2)
- TP5 pad 1: Net-(U13-INT3) -> Net-(U12-INT3)
- TP6 pad 1: Net-(U13-INT4) -> Net-(U12-INT4)
- U12 pad 1: GND -> Net-(U12-INT2)
- U12 pad 10: Net-(J9-Pin_5) -> GND
- U12 pad 11: Net-(J9-Pin_6) -> /+3.3v
- U12 pad 12: Net-(J9-Pin_7) -> Net-(U12-INT3)
- U12 pad 13: Net-(J9-Pin_8) -> Net-(U12-INT4)
- U12 pad 14: GND -> unconnected-(U12-CSB1-Pad14)
- U12 pad 15: Net-(J9-Pin_9) -> GND
- U12 pad 16: Net-(J9-Pin_10) -> Net-(U12-INT1)
- U12 pad 3: GND -> /+3.3v
- U12 pad 5: GND -> unconnected-(U12-CSB2-Pad5)
- U12 pad 6: /Sensors/LED0 -> GND
- U12 pad 7: Net-(J9-Pin_2) -> /+3.3v
- U12 pad 8: Net-(J9-Pin_3) -> /CM4_GPIO ( Ethernet, GPIO, SDCARD)/SCL0
- U12 pad 9: Net-(J9-Pin_4) -> /CM4_GPIO ( Ethernet, GPIO, SDCARD)/SDA0
- U9 pad 4: Net-(R12-Pad2) -> Net-(R14-Pad2)
Other:
- board outline added: 22 x 4 mm

Commit message: Feat: imported m.2 connector and more work on carrier board
Parts:
- removed J12: Conn_02x40_Odd_Even, M.2:NGFF_A
- added J11: 2199119-8, M.2_Connector:TE_2199119-8, F.Cu at (158.9, 57.8)
- moved J1 14.5 mm to (220.4, 110.1)
- moved J10 14.5 mm to (149.6, 156.1)
- moved J2 14.5 mm to (223.3, 74.9)
- moved J3 14.5 mm to (206.4, 90.1)
- moved J4 14.5 mm to (219.4, 92.5)
- moved U1 14.5 mm to (209.5, 110.4)
- moved U12 14.5 mm to (150.9, 142.9)
- moved U3 14.5 mm to (201.4, 98.6)
- moved Y1 14.5 mm to (201.6, 82.1)
- moved D20 14.5 mm to (-11.1, 74.7)
- moved D24 14.5 mm to (-11.1, 85.1)
- moved C10 14.5 mm to (-39.1, 98.6)
- moved C11 14.5 mm to (-39.1, 100.6)
- moved C12 14.5 mm to (-28.1, 101.1)
- moved C13 14.5 mm to (-39.1, 102.5)
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Other:
- board outline removed

Commit message: Refactor: updated to 4 layer pcb project
Parts:
- moved U1 7.66 mm to (205.1, 104.1)
- moved U12 7.66 mm to (146.5, 136.6)
- moved J11 7.66 mm to (154.5, 51.5)
- moved C17 7.66 mm to (-35.2, 81.1)
- moved C32 7.66 mm to (56.1, 70.8)
- moved C35 7.66 mm to (56.1, 78.4)
- moved C6 7.66 mm to (-35.2, 72.1)
- moved C8 7.66 mm to (-43.4, 88.4)
- moved C9 7.66 mm to (-43.4, 90.3)
- moved D2 7.66 mm to (33.3, 103.6)
- moved D20 7.66 mm to (-15.5, 68.4)
- moved D5 7.66 mm to (49.9, 74.5)
- moved D8 7.66 mm to (49.9, 94.3)
- moved J7 7.66 mm to (95.5, 119.7)
- moved JP2 7.66 mm to (12.7, 66.3)
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Other:
- copper layers 2 -> 4

Commit message: Feat: organized PCB file, preparing for layout and routing.
Parts:
- moved H1 276.4 mm to (253.5, 23.9)
- moved H2 276.4 mm to (253.5, 30.8)
- moved H3 276.4 mm to (260.4, 23.9)
- moved H4 276.4 mm to (260.4, 30.8)
- moved H5 276.4 mm to (267.4, 23.9)
- moved H6 276.4 mm to (267.4, 30.8)
- moved H7 276.4 mm to (274.3, 23.9)
- moved H8 276.4 mm to (274.3, 30.8)
- moved U5 248.2 mm to (207.3, 73.5)
- moved R10 243.9 mm to (197.5, 104.2)
- moved R9 243.9 mm to (197.5, 102.2)
- moved C3 239.4 mm to (195.5, 69.5)
- moved C7 239.4 mm to (195.5, 71.5)
- moved R3 238.8 mm to (192.4, 89.3)
- moved R4 238.8 mm to (192.4, 91.3)
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
Commit message: Feat: begun work on finalizing PCB layout
Parts:
- added J12: Conn_01x05, Connector_Molex:Molex_PicoBlade_53048-0510_1x05_P1.25mm_Horizontal, F.Cu at (137.3, 149.9)
- BZ1: moved to B.Cu
- Y1: footprint Crystal:Crystal_SMD_HC49-SD -> Crystal:Crystal_SMD_SeikoEpson_FA238-4Pin_3.2x2.5mm
- moved C32 193.0 mm to (65.0, 48.7)
- moved C35 193.0 mm to (72.6, 48.7)
- moved D5 193.0 mm to (68.7, 54.9)
- moved U15 193.0 mm to (101.3, 54.4)
- moved C30 193.0 mm to (60.0, 48.7)
- moved C33 193.0 mm to (67.5, 48.7)
- moved D4 193.0 mm to (62.1, 54.9)
- moved D8 193.0 mm to (88.5, 54.9)
- moved D9 193.0 mm to (95.2, 54.9)
- moved R20 193.0 mm to (75.1, 48.7)
- moved TP35 193.0 mm to (78.1, 48.9)
- moved C31 193.0 mm to (62.5, 48.7)
- moved C34 193.0 mm to (70.1, 48.7)
- moved D6 193.0 mm to (75.3, 54.9)
- moved D7 193.0 mm to (81.9, 54.9)
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Connections:
- J11 pad 1: /Connectors/RX -> /RX
- J11 pad 16: /Connectors/+5v -> /+5v
- J11 pad 18: /Connectors/+5v -> /+5v
- J11 pad 20: /Connectors/+5v -> /+5v
- J11 pad 22: /Connectors/+5v -> /+5v
- J11 pad 24: /Connectors/+5v -> /+5v
- J11 pad 26: /Connectors/+5v -> /+5v
- J11 pad 28: /Connectors/+5v -> /+5v
- J11 pad 3: /Connectors/RX -> /RX
- J11 pad 30: /Connectors/+5v -> /+5v
- J11 pad 32: /Connectors/+5v -> /+5v
- J11 pad 34: /Connectors/+5v -> /+5v
- J11 pad 36: /Connectors/+5v -> /+5v
- J11 pad 38: /Connectors/+5v -> /+5v
- J11 pad 40: /Connectors/+5v -> /+5v
- J11 pad 42: /Connectors/+5v -> /+5v
- J11 pad 44: /Connectors/+5v -> /+5v
- J11 pad 46: /Connectors/+5v -> /+5v
- J11 pad 48: /Connectors/+5v -> /+5v
- J11 pad 5: /Connectors/TX -> /TX
- J11 pad 50: /Connectors/+5v -> /+5v
- J11 pad 52: /Connectors/+5v -> /+5v
- J11 pad 54: /Connectors/+5v -> /+5v
- J11 pad 56: /Connectors/+5v -> /+5v
- J11 pad 58: /Connectors/+5v -> /+5v
- J11 pad 60: /Connectors/+5v -> /+5v
- J11 pad 62: /Connectors/+5v -> /+5v
- J11 pad 64: /Connectors/+5v -> /+5v
- J11 pad 66: /Connectors/+5v -> /+5v
- J11 pad 68: /Connectors/+5v -> /+5v
- J11 pad 7: /Connectors/TX -> /TX
- J11 pad 70: /Connectors/+5v -> /+5v
- J11 pad 72: /Connectors/+5v -> /+5v
- J11 pad 74: /Connectors/+5v -> /+5v
- J7 pad 10: /CM4_GPIO ( Ethernet, GPIO, SDCARD)/GPIO15 -> /TX
- J7 pad 8: /CM4_GPIO ( Ethernet, GPIO, SDCARD)/GPIO14 -> /RX
- Module1 pad 51: /CM4_GPIO ( Ethernet, GPIO, SDCARD)/GPIO15 -> /TX
- Module1 pad 55: /CM4_GPIO ( Ethernet, GPIO, SDCARD)/GPIO14 -> /RX
- Y1 pad 2: Net-(U3-XTALOUT) -> GND

Commit message: Feat: first draft pcb layout
Parts:
- removed H7, H8: MountingHole, MountingHole:MountingHole_2.7mm_M2.5
- BZ1: moved to F.Cu
- moved H2 148.5 mm to (154.6, 158.6)
- moved SW10 147.5 mm to (92.4, 168.4), turned to 90 degrees
- moved SW13 141.2 mm to (92.4, 160.4), turned to 90 degrees
- moved D19 140.7 mm to (96.6, 167.1), turned to -90 degrees
- moved SW11 135.7 mm to (102.9, 168.4), turned to 90 degrees
- moved SW16 135.5 mm to (92.4, 152.4), turned to 90 degrees
- moved D22 133.8 mm to (96.6, 158.7), turned to -90 degrees
- moved D20 129.5 mm to (107.0, 167.4), turned to -90 degrees
- moved SW14 128.8 mm to (102.9, 160.4), turned to 90 degrees
- moved D25 128.0 mm to (96.6, 150.9), turned to -90 degrees
- moved H3 127.7 mm to (82.2, 155.8)
- moved JP5 124.2 mm to (98.7, 147.1), turned to 90 degrees
- moved SW12 123.5 mm to (114.5, 168.4), turned to 90 degrees
- moved SW17 122.6 mm to (102.9, 152.4), turned to 90 degrees
- moved D23 122.0 mm to (107.0, 159.0), turned to -90 degrees
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Connections:
- D6 pad 1: unconnected-(D6-VDD-Pad1) -> /+5v
- D7 pad 1: unconnected-(D7-VDD-Pad1) -> /+5v
- D8 pad 1: unconnected-(D8-VDD-Pad1) -> /+5v
- D9 pad 1: unconnected-(D9-VDD-Pad1) -> /+5v
Other:
- board outline added: 82 x 162.1 mm
- board text added: "POWER BOARD"

Commit message: Feat: progress routing usb and hdmi
Parts:
- moved C17 64.5 mm to (181.0, 47.7)
- moved C14 64.5 mm to (175.0, 47.7)
- moved C18 64.5 mm to (184.0, 47.7)
- moved C4 64.5 mm to (177.8, 51.5)
- moved C12 64.5 mm to (187.1, 54.2)
- moved C16 64.5 mm to (178.0, 47.7)
- moved R9 33.0 mm to (142.5, 36.3), turned to -45 degrees
- moved J3 30.9 mm to (117.5, 32.9), turned to -90 degrees
- moved C5 26.5 mm to (111.2, 47.4)
- moved C6 26.5 mm to (111.3, 49.8)
- moved C10 26.5 mm to (107.1, 48.6)
- moved C11 26.5 mm to (107.1, 50.6)
- moved C13 26.5 mm to (107.1, 52.6)
- moved C15 26.5 mm to (107.1, 54.5)
- moved C8 26.5 mm to (107.1, 44.7)
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Routing:
- net /CM4_HighSpeed/HDMI0_D2_P: track 0.00 -> 39.2 mm
- net /CM4_HighSpeed/HDMI0_D2_N: track 0.00 -> 39.2 mm
- net /CM4_HighSpeed/HDMI0_D1_P: track 0.00 -> 37.2 mm
- net /CM4_HighSpeed/HDMI0_D1_N: track 0.00 -> 37.2 mm
- net /CM4_HighSpeed/HDMI0_D0_P: track 0.00 -> 35.2 mm
- net /CM4_HighSpeed/HDMI0_D0_N: track 0.00 -> 34.4 mm
- net /CM4_HighSpeed/HDMI0_CK_P: track 0.00 -> 33.2 mm
- net /CM4_HighSpeed/HDMI0_CK_N: track 0.00 -> 33.1 mm
- net Net-(JP4-A): track 0.00 -> 26.3 mm
- net Net-(JP3-A): track 0.00 -> 25.6 mm
- net Net-(JP2-A): track 0.00 -> 25.4 mm
- net /USB2-HUB/USBD_P: track 0.00 -> 24.8 mm
- net /USB2-HUB/USBD_N: track 0.00 -> 24.6 mm
- net /USB2-HUB/HD4_P: track 0.00 -> 22.0 mm
- net /USB2-HUB/HD4_N: track 0.00 -> 21.9 mm
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- added copper zone on F.Cu, net /+5v
- added copper zone on B.Cu, net GND
- added copper zone on F.Cu, net GND
- added copper zone on In1.Cu, net GND
- added copper zone on In2.Cu, net GND
