File: esc/rp2040_module/rp2040_module.kicad_pcb (KiCad board)
At the start: 0 parts

Commit message: Feat[esc]: schematic to pcb placement of B-G431B-ESC1 + RP2040
Parts:
- added C1: 0.1uF, Capacitor_SMD:C_0402_1005Metric, F.Cu at (194.6, 109.5)
- added C10: 0.1uF, Capacitor_SMD:C_0402_1005Metric, F.Cu at (198.6, 102.3)
- added C11: 1uF, Capacitor_SMD:C_0402_1005Metric, F.Cu at (205.2, 102.4)
- added C12: 27pF, Capacitor_SMD:C_0402_1005Metric, F.Cu at (200.1, 115.3)
- added C13: 27pF, Capacitor_SMD:C_0402_1005Metric, F.Cu at (195.7, 114.5)
- added C14: 1uF, Capacitor_SMD:C_0402_1005Metric, F.Cu at (189.0, 97.5)
- added C2: 0.1uF, Capacitor_SMD:C_0402_1005Metric, F.Cu at (199.6, 102.3)
- added C3: 0.1uF, Capacitor_SMD:C_0402_1005Metric, F.Cu at (200.8, 113.8)
- added C4: 0.1uF, Capacitor_SMD:C_0402_1005Metric, F.Cu at (200.7, 102.3)
- added C5: 0.1uF, Capacitor_SMD:C_0402_1005Metric, F.Cu at (205.0, 104.8)
- added C6: 0.1uF, Capacitor_SMD:C_0402_1005Metric, F.Cu at (205.0, 109.5)
- added C7: 0.1uF, Capacitor_SMD:C_0402_1005Metric, F.Cu at (194.6, 105.9)
- added C8: 0.1uF, Capacitor_SMD:C_0402_1005Metric, F.Cu at (201.9, 113.8)
- added C9: 1uF, Capacitor_SMD:C_0402_1005Metric, F.Cu at (206.2, 102.4)
- added J1: USB_C_Receptacle_USB2.0, Connector_USB:USB_C_Receptacle_HRO_TYPE-C-31-M-12, F.Cu at (201.9, 95.7)
- added J2: Conn_01x04, Connector_PinHeader_2.54mm:PinHeader_1x04_P2.54mm_Vertical, F.Cu at (186.7, 94.9)
- added J3: 5530843-7, 5530843-7_PCB_Edge:TE_5530843-7_PCB_Edge, F.Cu at (169.9, 130.0)
- added R1: 10K, Resistor_SMD:R_0402_1005Metric, F.Cu at (203.4, 114.0)
- added R2: 5.1k, Resistor_SMD:R_0402_1005Metric, F.Cu at (195.3, 98.0)
- added R3: 5.1k, Resistor_SMD:R_0402_1005Metric, F.Cu at (194.3, 98.0)
- added R4: 27, Resistor_SMD:R_0603_1608Metric, F.Cu at (202.2, 102.6)
- added R5: 27, Resistor_SMD:R_0603_1608Metric, F.Cu at (203.8, 102.6)
- added R6: 1K, Resistor_SMD:R_0402_1005Metric, F.Cu at (199.6, 113.8)
- added R7: 1K, Resistor_SMD:R_0402_1005Metric, F.Cu at (192.5, 104.6)
- added R8: 10K, Resistor_SMD:R_0402_1005Metric, F.Cu at (190.2, 104.6)
- added SW1: SW_Push, SLIM_6MM_Switch:SW_PUSH_6mm_SLIM, F.Cu at (187.6, 107.1)
- added SW2: SW_Push, SLIM_6MM_Switch:SW_PUSH_6mm_SLIM, F.Cu at (191.1, 107.1)
- added U1: RP2040, Package_DFN_QFN:QFN-56-1EP_7x7mm_P0.4mm_EP3.2x3.2mm_ThermalVias, F.Cu at (199.7, 108.5)
- added U2: W25Q64JVXGIQ, Package_SO:SOIC-8_5.23x5.23mm_P1.27mm, F.Cu at (188.2, 101.0)
- added U3: B-G431B-ESC1, B-G431B-ESC1:B-G431B-ESC1_MOUNT, F.Cu at (156.7, 106.6)
- added Y1: 12MHz, Crystal:Crystal_SMD_2016-4Pin_2.0x1.6mm, F.Cu at (197.7, 114.7)
Other:
- board outline added: 78.4 x 29.7 mm
- copper layers 0 -> 2
