File: breakouts/bme680/bme680.kicad_sch (KiCad schematic)
At the start: 7 parts, among them J1 Conn_01x04, J2 Conn_01x02, U1 BME680

Commit message: Feat[leds]: added power leds to breakouts
Parts:
- added D1: PWR, LED_SMD:LED_0603_1608Metric, symbol Device:LED_Small
- added R1: 10k, Resistor_SMD:R_0603_1608Metric, symbol Device:R_Small
Connections:
- net +3.3V: now also R1.1
- net GND: now also D1.1 (K)
- new net: D1.2 (A), R1.2
Changed lines of the file:
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@@
+    )
+  )
+  (symbol (lib_id "Device:R_Small") (at 86.36 100.33 0) (unit 1)
+    (in_bom yes) (on_board yes) (dnp no) (fields_autoplaced)
+    (property "Reference" "R1" (at 88.9 99.695 0)
+      (effects (font (size 1.27 1.27)) (justify left))
+    )
+    (property "Value" "10k" (at 88.9 102.235 0)
+      (effects (font (size 1.27 1.27)) (justify left))
+    )
+    (property "Footprint" "Resistor_SMD:R_0603_1608Metric" (at 86.36 100.33 0)
+      (effects (font (size 1.27 1.27)) hide)
+    )
+    (property "Datasheet" "~" (at 86.36 100.33 0)
+      (effects (font (size 1.27 1.27)) hide)
+    )
+    (pin "1")
+    (pin "2")
+    (instances
+      (project "bmi088"
+        (path "/62de48e5-2947-447b-a8d0-ed636dc1e73b"
+          (reference "R1") (unit 1)
+        )
+      )
+      (project "bme680"
+        (path "/81348711-088d-4268-b70f-3c2090b69805"
+          (reference "R1") (unit 1)
+        )
+      )
     )
   )
@@
         (path "/81348711-088d-4268-b70f-3c2090b69805"
           (reference "JP1") (unit 1)
+        )
+      )
+    )
+  )
+  (symbol (lib_id "power:GND") (at 86.36 107.95 0) (unit 1)
+    (in_bom yes) (on_board yes) (dnp no) (fields_autoplaced)
+    (property "Reference" "#PWR09" (at 86.36 114.3 0)
+      (effects (font (size 1.27 1.27)) hide)
+    )
+    (property "Value" "GND" (at 86.36 113.03 0)
+      (effects (font (size 1.27 1.27)))
+    )
+    (property "Footprint" "" (at 86.36 107.95 0)
+      (effects (font (size 1.27 1.27)) hide)
+    )
+    (property "Datasheet" "" (at 86.36 107.95 0)
+      (effects (font (size 1.27 1.27)) hide)
+    )
+    (pin "1")
+    (instances
+      (project "bmi088"
+        (path "/62de48e5-2947-447b-a8d0-ed636dc1e73b"
+          (reference "#PWR09") (unit 1)
+        )
+      )
+      (project "bme680"
+        (path "/81348711-088d-4268-b70f-3c2090b69805"
+          (reference "#PWR09") (unit 1)
         )
       )
@@
     )
   )
+  (symbol (lib_id "power:+3.3V") (at 86.36 97.79 0) (unit 1)
+    (in_bom yes) (on_board yes) (dnp no) (fields_autoplaced)
+    (property "Reference" "#PWR010" (at 86.36 101.6 0)
+      (effects (font (size 1.27 1.27)) hide)
+    )
+    (property "Value" "+3.3V" (at 86.36 93.98 0)
+      (effects (font (size 1.27 1.27)))
+    )
+    (property "Footprint" "" (at 86.36 97.79 0)
+      (effects (font (size 1.27 1.27)) hide)
+    )
+    (property "Datasheet" "" (at 86.36 97.79 0)
+      (effects (font (size 1.27 1.27)) hide)
+    )
+    (pin "1")
+    (instances
+      (project "bmi088"
+        (path "/62de48e5-2947-447b-a8d0-ed636dc1e73b"
+          (reference "#PWR010") (unit 1)
+        )
+      )
+      (project "bme680"
+        (path "/81348711-088d-4268-b70f-3c2090b69805"
+          (reference "#PWR08") (unit 1)
+        )
+      )
+    )
+  )
   (symbol (lib_id "power:+3.3V") (at 160.02 106.68 0) (unit 1)
     (in_bom yes) (on_board yes) (dnp no) (fields_autoplaced)
@@
         )
       )
+    )
+  )
+  (symbol (lib_id "Device:LED_Small") (at 86.36 105.41 90) (unit 1)
+    (in_bom yes) (on_board yes) (dnp no) (fields_autoplaced)
+    (property "Reference" "D1" (at 88.9 104.7115 90)
+      (effects (font (size 1.27 1.27)) (justify right))
+    )
+    (property "Value" "PWR" (at 88.9 107.2515 90)
+      (effects (font (size 1.27 1.27)) (justify right))
+    )
+    (property "Footprint" "LED_SMD:LED_0603_1608Metric" (at 86.36 105.41 90)
+      (effects (font (size 1.27 1.27)) hide)
+    )
+    (property "Datasheet" "~" (at 86.36 105.41 90)
+      (effects (font (size 1.27 1.27)) hide)
+    )
+    (pin "1")
+    (pin "2")
+    (instances
+      (project "bmi088"
+        (path "/62de48e5-2947-447b-a8d0-ed636dc1e73b"
+          (reference "D1") (unit 1)
+        )
+      )
+      (project "bme680"
+        (path "/81348711-088d-4268-b70f-3c2090b69805"
+          (reference "D1") (unit 1)
+        )
+      )
