File: networking/switch/magnetics.kicad_sch (KiCad schematic)
At the start: 20 parts, among them J3 PHY 5, J4 PHY 4, J5 PHY 3, J6 PHY 2, J7 PHY 1, T1 Dual Transformer, T2 Dual Transformer, U4 Single Transformer

Commit message: Feat[switch]: created all necessary symbols and footprints, started PCB
Parts:
- C24, C25, C26, C27, C28: footprint (none) -> Capacitor_SMD:C_0402_1005Metric
- C29, C30: footprint (none) -> Capacitor_SMD:C_1206_3216Metric
- J3, J4, J5, J6, J7: footprint (none) -> Connector_Molex:Molex_PicoBlade_53398-0471_1x04-1MP_P1.25mm_Vertical
- R21, R22, R23, R24, R25: footprint (none) -> Resistor_SMD:R_0402_1005Metric
- T1, T2: footprint (none) -> QT24A23:QT24A23
- U4: footprint (none) -> BT16A07:BT16A07
Changed lines of the file:
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@@
       (effects (font (size 1.27 1.27)) (justify left))
     )
-    (property "Footprint" "" (at 81.28 137.16 0)
+    (property "Footprint" "Capacitor_SMD:C_0402_1005Metric" (at 81.28 137.16 0)
       (effects (font (size 1.27 1.27)) hide)
     )
@@
       (effects (font (size 1.27 1.27)) (justify left))
     )
-    (property "Footprint" "" (at 180.34 58.42 0)
+    (property "Footprint" "Capacitor_SMD:C_1206_3216Metric" (at 180.34 58.42 0)
       (effects (font (size 1.27 1.27)) hide)
     )
@@
       (effects (font (size 1.27 1.27)) (justify left))
     )
-    (property "Footprint" "" (at 181.61 143.51 0)
+    (property "Footprint" "Capacitor_SMD:C_1206_3216Metric" (at 181.61 143.51 0)
       (effects (font (size 1.27 1.27)) hide)
     )
@@
       (effects (font (size 1.27 1.27)))
     )
-    (property "Footprint" "" (at 149.86 130.81 0)
+    (property "Footprint" "Resistor_SMD:R_0402_1005Metric" (at 149.86 130.81 0)
       (effects (font (size 1.27 1.27)) hide)
     )
@@
       (effects (font (size 1.27 1.27)) (justify left))
     )
-    (property "Footprint" "" (at 81.28 55.88 0)
+    (property "Footprint" "Capacitor_SMD:C_0402_1005Metric" (at 81.28 55.88 0)
       (effects (font (size 1.27 1.27)) hide)
     )
@@
       (effects (font (size 1.27 1.27)) (justify left))
     )
-    (property "Footprint" "" (at 218.44 73.66 0)
+    (property "Footprint" "Connector_Molex:Molex_PicoBlade_53398-0471_1x04-1MP_P1.25mm_Vertical" (at 218.44 73.66 0)
       (effects (font (size 1.27 1.27)) hide)
     )
@@
       (effects (font (size 1.27 1.27)))
     )
-    (property "Footprint" "" (at 133.35 137.16 0)
+    (property "Footprint" "QT24A23:QT24A23" (at 133.35 137.16 0)
       (effects (font (size 1.27 1.27)) hide)
     )
@@
       (effects (font (size 1.27 1.27)))
     )
-    (property "Footprint" "" (at 149.86 87.63 0)
+    (property "Footprint" "Resistor_SMD:R_0402_1005Metric" (at 149.86 87.63 0)
       (effects (font (size 1.27 1.27)) hide)
     )
@@
       (effects (font (size 1.27 1.27)))
     )
-    (property "Footprint" "" (at 149.86 142.24 0)
+    (property "Footprint" "Resistor_SMD:R_0402_1005Metric" (at 149.86 142.24 0)
       (effects (font (size 1.27 1.27)) hide)
     )
@@
       (effects (font (size 1.27 1.27)) (justify left))
     )
-    (property "Footprint" "" (at 95.25 137.16 0)
+    (property "Footprint" "Capacitor_SMD:C_0402_1005Metric" (at 95.25 137.16 0)
       (effects (font (size 1.27 1.27)) hide)
     )
@@
       (effects (font (size 1.27 1.27)) (justify left))
     )
-    (property "Footprint" "" (at 218.44 107.95 0)
+    (property "Footprint" "Connector_Molex:Molex_PicoBlade_53398-0471_1x04-1MP_P1.25mm_Vertical" (at 218.44 107.95 0)
       (effects (font (size 1.27 1.27)) hide)
     )
@@
       (effects (font (size 1.27 1.27)) (justify left))
     )
-    (property "Footprint" "" (at 81.28 91.44 0)
+    (property "Footprint" "Capacitor_SMD:C_0402_1005Metric" (at 81.28 91.44 0)
       (effects (font (size 1.27 1.27)) hide)
     )
@@
       (effects (font (size 1.27 1.27)))
     )
-    (property "Footprint" "" (at 149.86 99.06 0)
+    (property "Footprint" "Resistor_SMD:R_0402_1005Metric" (at 149.86 99.06 0)
       (effects (font (size 1.27 1.27)) hide)
     )
@@
       (effects (font (size 1.27 1.27)))
     )
-    (property "Footprint" "" (at 133.35 57.15 0)
+    (property "Footprint" "BT16A07:BT16A07" (at 133.35 57.15 0)
       (effects (font (size 1.27 1.27)) hide)
     )
@@
       (effects (font (size 1.27 1.27)))
     )
-    (property "Footprint" "" (at 133.35 93.98 0)
+    (property "Footprint" "QT24A23:QT24A23" (at 133.35 93.98 0)
       (effects (font (size 1.27 1.27)) hide)
     )
@@
       (effects (font (size 1.27 1.27)) (justify left))
     )
-    (property "Footprint" "" (at 218.44 96.52 0)
+    (property "Footprint" "Connector_Molex:Molex_PicoBlade_53398-0471_1x04-1MP_P1.25mm_Vertical" (at 218.44 96.52 0)
       (effects (font (size 1.27 1.27)) hide)
     )
@@
       (effects (font (size 1.27 1.27)) (justify left))
     )
-    (property "Footprint" "" (at 180.34 53.34 0)
+    (property "Footprint" "Resistor_SMD:R_0402_1005Metric" (at 180.34 53.34 0)
       (effects (font (size 1.27 1.27)) hide)
     )
@@
       (effects (font (size 1.27 1.27)) (justify left))
     )
-    (property "Footprint" "" (at 218.44 62.23 0)
+    (property "Footprint" "Connector_Molex:Molex_PicoBlade_53398-0471_1x04-1MP_P1.25mm_Vertical" (at 218.44 62.23 0)
       (effects (font (size 1.27 1.27)) hide)
     )
@@
       (effects (font (size 1.27 1.27)) (justify left))
     )
-    (property "Footprint" "" (at 218.44 85.09 0)
+    (property "Footprint" "Connector_Molex:Molex_PicoBlade_53398-0471_1x04-1MP_P1.25mm_Vertical" (at 218.44 85.09 0)
       (effects (font (size 1.27 1.27)) hide)
     )
@@
       (effects (font (size 1.27 1.27)) (justify left))
     )
-    (property "Footprint" "" (at 95.25 91.44 0)
-      (effects (font (size 1.27 1.27)) hide)
-    )
+    (property "Footprint" "Capacitor_SMD:C_0402_1005Metric" (at 95.25 91.44 0)
+      (effects (font (size 1.27 1.27)) hide)
+    )

Commit message: Feat[switch]: initial board layout (FOLLOW @TODOs)
Parts:
- removed T1: Dual Transformer, QT24A23:QT24A23, symbol magnetics:dual-transformer
- added C31, C32, C33: 1nF 2KV (1206), Capacitor_SMD:C_1206_3216Metric, symbol Device:C_Small
- added T1: QT24A23-ALT, QT24A23:QT24A23, symbol magnetics:dual-transformer-2
- J4: renamed from J3; footprint Connector_Molex:Molex_PicoBlade_53398-0471_1x04-1MP_P1.25mm_Vertical -> Connector_Molex:Molex_PicoBlade_53047-0410_1x04_P1.25mm_Vertical
- J5: renamed from J4; footprint Connector_Molex:Molex_PicoBlade_53398-0471_1x04-1MP_P1.25mm_Vertical -> Connector_Molex:Molex_PicoBlade_53047-0410_1x04_P1.25mm_Vertical
- J6: renamed from J5; footprint Connector_Molex:Molex_PicoBlade_53398-0471_1x04-1MP_P1.25mm_Vertical -> Connector_Molex:Molex_PicoBlade_53047-0410_1x04_P1.25mm_Vertical
- J7: renamed from J6; footprint Connector_Molex:Molex_PicoBlade_53398-0471_1x04-1MP_P1.25mm_Vertical -> Connector_Molex:Molex_PicoBlade_53047-0410_1x04_P1.25mm_Vertical
- J8: renamed from J7; footprint Connector_Molex:Molex_PicoBlade_53398-0471_1x04-1MP_P1.25mm_Vertical -> Connector_Molex:Molex_PicoBlade_53047-0410_1x04_P1.25mm_Vertical
- T2: value Dual Transformer -> QT24A23
- U4: value Single Transformer -> BT16A07
Connections:
- net CT0: now also T2.10 (CT1), T2.7 (CT1); no longer T2.8 (CT1)
- net CT1: now also T2.1 (CT2), T2.4 (CT2); no longer T2.3 (CT2)
- net CT2: now also T1.10 (CT1), T1.7 (CT1)
- net CT3: now also T1.1 (CT2), T1.4 (CT2)
- net CT4: no longer U4.5 (CT)
- net Earth: now also C31.2, C32.2, C33.2
- net REF0: no longer R21.2, R22.2, R23.2
- net REF4: no longer U4.13 (MCT)
- net RX0+: now also J8.1 (Pin_1), T2.13 (RX1+); no longer J8.3 (Pin_3), T2.11 (RX1+), T2.14 (TX1+)
- net RX0-: now also J8.2 (Pin_2), T2.14 (RX1-); no longer J8.4 (Pin_4), T2.12 (RX1-)
- net RX1+: now also J7.1 (Pin_1), T2.23 (RX2+); no longer J7.3 (Pin_3), T2.20 (RX2+)
- net RX1-: now also J7.2 (Pin_2), T2.22 (RX2-); no longer J7.4 (Pin_4), T2.19 (RX2-)
- net RX2+: now also J6.1 (Pin_1), T1.13 (RX1+); no longer J6.3 (Pin_3)
- net RX2-: now also J6.2 (Pin_2), T1.14 (RX1-); no longer J6.4 (Pin_4)
- net RX3+: now also J5.1 (Pin_1), T1.19 (TX2+); no longer J5.3 (Pin_3)
- net RX3-: now also J5.2 (Pin_2), T1.20 (TX2-); no longer J5.4 (Pin_4)
- net RX4+: now also J4.1 (Pin_1); no longer J4.3 (Pin_3)
- net RX4-: now also J4.2 (Pin_2); no longer J4.4 (Pin_4)
- net RXIM0: now also T2.11 (RD1-); no longer T2.9 (RD1-)
- net RXIM1: now also T2.3 (RD2-); no longer T2.2 (RD2-)
- net RXIM2: now also T1.11 (RD1-)
- net RXIM3: now also T1.5 (TD2-)
- net RXIP0: now also T2.12 (RD1+); no longer T2.10 (RD1+)
- net RXIP1: now also T2.2 (RD2+); no longer T2.1 (RD2+)
- net RXIP2: now also T1.12 (RD1+)
- net RXIP3: now also T1.6 (TD2+)
- net TX0+: now also J8.3 (Pin_3), T2.16 (TX1+); no longer J8.1 (Pin_1)
- net TX0-: now also J8.4 (Pin_4), T2.17 (TX1-); no longer J8.2 (Pin_2), T2.15 (TX1-)
- net TX1+: now also J7.3 (Pin_3), T2.20 (TX2+); no longer J7.1 (Pin_1), T2.17 (TX2+)
- net TX1-: now also J7.4 (Pin_4), T2.19 (TX2-); no longer J7.2 (Pin_2), T2.16 (TX2-)
- net TX2+: now also J6.3 (Pin_3), T1.16 (TX1+); no longer J6.1 (Pin_1)
- net TX2-: now also J6.4 (Pin_4), T1.17 (TX1-); no longer J6.2 (Pin_2)
- net TX3+: now also J5.3 (Pin_3), T1.22 (RX2+); no longer J5.1 (Pin_1)
- net TX3-: now also J5.4 (Pin_4), T1.23 (RX2-); no longer J5.2 (Pin_2)
- net TX4+: now also J4.3 (Pin_3); no longer J4.1 (Pin_1)
- net TX4-: now also J4.4 (Pin_4); no longer J4.2 (Pin_2)
- net TXOM0: now also T2.8 (TD1-); no longer T2.6 (TD1-)
- net TXOM1: now also T2.6 (TD2-); no longer T2.5 (TD2-)
- net TXOM2: now also T1.8 (TD1-)
- net TXOM3: now also T1.2 (RD2-)
- net TXOP0: now also T2.9 (TD1+); no longer T2.7 (TD1+)
- net TXOP1: now also T2.5 (TD2+); no longer T2.4 (TD2+)
- net TXOP2: now also T1.9 (TD1+)
- net TXOP3: now also T1.3 (RD2+)
- net at R23.1: now also T2.21 (CMG2), T2.24 (CMG2); no longer T2.18 (CMG0)
- net at R24.1: now also T2.15 (CMG1), T2.18 (CMG1); no longer T2.13 (CMG1)
- net at R21.1: now also T1.21 (CMG2), T1.24 (CMG2)
- net at R22.1: now also T1.15 (CMG1), T1.18 (CMG1)
- new net REF1: C33.1, R23.2
- new net REF2: C31.1, R22.2
- new net REF3: C32.1, R21.2
- no-connect marks 2 -> 4
Other:
- note added: "Pinout: RX+, RX-, TX+, TX-"
- note removed: "Pinout: TX+, TX-, RX+, RX-"
- moved on the sheet: R21, R22, R23, R24
