File: SID/usb_camera.kicad_sch (KiCad schematic)
At the start: 0 parts

Commit message: Feat(SID): basically complete
Changed lines of the file:
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@@
 	(generator_version "8.99")
 	(paper "A4")
-	(hierarchical_label "Phases IN"
-		(shape bidirectional)
-		(at 109.22 99.06 0)
+	(hierarchical_label "USB"
+		(shape input)
+		(at 109.22 85.09 0)
 		(fields_autoplaced yes)
 		(effects
