File: power/TPS568230.kicad_sch (KiCad schematic)
At the start: 24 parts, among them U1 TPS568230RJER

Commit message: Feat[power]: initial layout
Parts:
- removed TP1: 5V, TestPoint:TestPoint_Pad_1.5x1.5mm, symbol Connector:TestPoint
Changed lines of the file:
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@@
-    (stroke (width 0) (type default))
-  )
-  (wire (pts (xy 188.976 89.154) (xy 188.976 90.424))
     (stroke (width 0) (type default))
   )
@@
         )
       )
-    )
-  )
-  (symbol (lib_id "Connector:TestPoint") (at 188.976 89.154 0) (unit 1)
-    (exclude_from_sim no) (in_bom yes) (on_board yes) (dnp no) (fields_autoplaced)
-    (property "Reference" "TP1" (at 191.262 84.582 0)
-      (effects (font (size 1.27 1.27)) (justify left))
-    )
-    (property "Value" "5V" (at 191.262 87.122 0)
-      (effects (font (size 1.27 1.27)) (justify left))
-    )
-    (property "Footprint" "TestPoint:TestPoint_Pad_1.5x1.5mm" (at 194.056 89.154 0)
-      (effects (font (size 1.27 1.27)) hide)
-    )
-    (property "Datasheet" "~" (at 194.056 89.154 0)
-      (effects (font (size 1.27 1.27)) hide)
-    )
-    (property "Description" "test point" (at 188.976 89.154 0)
-      (effects (font (size 1.27 1.27)) hide)
-    )
-    (pin "1")
-    (instances
-      (project "power"
-        (path "/6d3c5c52-febb-4c99-82d7-f9b22bb5762b/e479a492-f085-4afe-886c-479f29421304"
-          (reference "TP1") (unit 1)
-        )
-      )

Commit message: Feat[power]: component mapping
Parts:
- C13: value 0.1uF -> 1uF
- R8: value 26.6k -> 27k
Changed lines of the file:
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@@
       (effects (font (size 1.27 1.27)) (justify left))
     )
-    (property "Value" "26.6k" (at 250.19 103.886 0)
+    (property "Value" "27k" (at 250.19 103.886 0)
       (effects (font (size 1.27 1.27)) (justify left))
     )
@@
   (symbol (lib_id "Device:R_Small") (at 145.542 98.044 0) (unit 1)
     (exclude_from_sim no) (in_bom yes) (on_board yes) (dnp no) (fields_autoplaced)
-    (property "Reference" "R4" (at 148.082 96.774 0)
-      (effects (font (size 1.27 1.27)) (justify left))
-    )
-    (property "Value" "226k" (at 148.082 99.314 0)
+    (property "Reference" "R4" (at 147.32 96.774 0)
+      (effects (font (size 1.27 1.27)) (justify left))
+    )
+    (property "Value" "226k" (at 147.32 99.314 0)
       (effects (font (size 1.27 1.27)) (justify left))
     )
@@
       (effects (font (size 1.27 1.27)) (justify left))
     )
-    (property "Value" "0.1uF" (at 242.062 85.09 0)
-      (effects (font (size 1.27 1.27)) (justify left))
-    )
+    (property "Value" "1uF" (at 242.062 85.09 0)
+      (effects (font (size 1.27 1.27)) (justify left))
+    )
