File: Smart Power Board/RP2040.kicad_sch (KiCad schematic)
At the start: 41 parts, among them J2 USB_C_Receptacle_USB2.0_16P, J3 Conn_01x04, Q1 PMOS, Q2 NMOS, SW1 SW_Push, SW2 SW_Push, U2 X096-2864TMBAG01-H30, U6 RP2040, U7 W25Q32JVSS, X1 ABM8-272-T3

Commit message: Feat[SmartPowerBoard]: Mid-Progress Update
Parts:
- removed R36: 10k, Resistor_SMD:R_0402_1005Metric, symbol Device:R_Small
- removed X1: ABM8-272-T3, ABM8-272-T3_ABR, symbol ABM8-272-T3:ABM8-272-T3
- added SW3: SW_Push, Button_Switch_SMD:SW_Push_SPST_NO_Alps_SKRK, symbol Switch:SW_Push
- added Y1: FL1200138, FL1200138:XTAL_FL1200138, symbol FL1200138:FL1200138
- C18: value 4.7uF -> 2.2uF
- C33, C34: footprint Capacitor_SMD:C_0201_0603Metric -> Capacitor_SMD:C_0402_1005Metric
- Q1: footprint IRF7416TRPBF_KiCad:SOIC127P600X175-8N -> FDN338P:SSOT-3
- Q2: footprint FDS6690A_KiCad:SOIC127P600X175-8N -> FDN335N:SSOT-3
Connections:
- net GND: now also C33.2, Q2.3 (S), R18.2, SW3.1, Y1.2 (GND), Y1.4 (GND__1); no longer C33.1
- net RES#: now also SW3.2
- net XIN: now also Y1.1
- net at R19.1: now also C33.1, Y1.3; no longer C33.2
- net ADC0: no longer names the net of U6.38 (GPIO26_ADC0)
- net ADC1: no longer names the net of U6.39 (GPIO27_ADC1)
- net ADC2: no longer names the net of U6.40 (GPIO28_ADC2)
- net ADC3: no longer names the net of U6.41 (GPIO29_ADC3)
- net OS: no longer names the net of U6.9 (GPIO7)
- no-connect marks 22 -> 27
Other:
- note added: "RES#"
- moved on the sheet: C33, C34, Q1, Q2, R12, R18, R19

Commit message: Feat[SmartPowerBoard]: New Layout
Parts:
- removed J3: Conn_01x04, Connector_PinHeader_2.54mm:PinHeader_1x04_P2.54mm_Vertical, symbol Connector_Generic:Conn_01x04
Connections:
- net SWCLK: no longer names the net of U6.24 (SWCLK)
- net SWD: no longer names the net of U6.25 (SWD)
- no-connect marks 27 -> 29
Other:
- note removed: "SWD Connection"

Commit message: Feat[SmartPowerBoard]: Organized Schematic and New Buck
Parts:
- removed C17, C19, C20: 4.7uF, Capacitor_SMD:C_0402_1005Metric, symbol Device:C_Small
- removed C18: 2.2uF, Capacitor_SMD:C_0402_1005Metric, symbol Device:C_Small
- removed C32, C36: 1uF, Capacitor_SMD:C_0402_1005Metric, symbol Device:C_Small
- removed Q1: PMOS, FDN338P:SSOT-3, symbol Simulation_SPICE:PMOS
- removed Q2: NMOS, FDN335N:SSOT-3, symbol Simulation_SPICE:NMOS
- removed R12, R18: 47k, Resistor_SMD:R_0402_1005Metric, symbol Device:R_Small
- removed R9: 620k, Resistor_SMD:R_0603_1608Metric_Pad0.98x0.95mm_HandSolder, symbol Device:R_Small
- removed SW3: SW_Push, Button_Switch_SMD:SW_Push_SPST_NO_Alps_SKRK, symbol Switch:SW_Push
- removed U2: X096-2864TMBAG01-H30, LIB_X096-2864TMBAG01-H30:X096-2864TMBAG01-H30, symbol New_Library:X096-2864TMBAG01-H30
Connections:
- net SCL: now also R37.2, U6.2 (GPIO0); no longer R38.2, U6.3 (GPIO1)
- net SDA: now also R38.2, U6.3 (GPIO1); no longer R37.2, U6.2 (GPIO0)
- net 3.3V renamed 3.3V_{CC}
- net 5V renamed 5V_{IN}
- no-connect marks 29 -> 28
Other:
- note removed: "Electronic Switch"
- note removed: "Main Display"
- note removed: "RES#"
- moved on the sheet: R34, R35, R37, R38

Commit message: Feat[SmartPowerBoard]: Internal Power + OLED
Connections:
- net GPIO4: now reaches U6.6 (GPIO4)
- no-connect marks 28 -> 27
Other:
- note removed: "OLED Display"
Changed lines of the file:
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@@
-	)
-	(no_connect
-		(at 90.17 99.06)
 	)
 	(no_connect
@@
 		(pts
 			(xy 90.17 88.9) (xy 93.98 88.9)
+		)
+		(stroke
+			(width 0)
+			(type default)
+		)
+	)
+	(wire
+		(pts
+			(xy 90.17 99.06) (xy 106.68 99.06)
 		)
 		(stroke
@@
 	)
 	(rectangle
-		(start 179.324 16.51)
-		(end 284.226 164.846)
-		(stroke
-			(width 0)
-			(type dash)
-		)
-		(fill
-			(type none)
-		)
-	)
-	(rectangle
 		(start 14.478 51.435)
 		(end 119.126 186.436)
@@
 		)
 	)
-	(text "OLED Display\n"
-		(exclude_from_sim no)
-		(at 187.706 20.32 0)
-		(effects
-			(font
-				(face "JetBrains Mono")
-				(size 1.27 1.27)
-			)
-		)
-	)
 	(text "USB_BOOT Button"
 		(exclude_from_sim no)
@@
 		(fields_autoplaced yes)
 		(effects
+			(font
+				(size 1.27 1.27)
+			)
+			(justify right bottom)
+		)
+	)
+	(label "GPIO4"
+		(at 106.68 99.06 180)
+		(fields_autoplaced yes)
+		(effects

Commit message: Feat[SmartPowerBoard]: Routing
Parts:
- added C36, C37, C38, C39, C40: 0.1uF, Capacitor_SMD:C_0402_1005Metric, symbol Device:C_Small
Connections:
- net 3.3V_{CC}: now also C36.2, C37.2, C38.2, C39.2, C40.2
- net GND: now also C36.1, C37.1, C38.1, C39.1, C40.1
- net RUN: now also R39.2, U6.26 (RUN)
Other:
- moved on the sheet: C13, C15, C16

Commit message: Feat[SmartPowerBoard]: More Routing
Changed lines of the file:
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@@
 	(wire
 		(pts
-			(xy 166.37 29.21) (xy 154.94 29.21)
+			(xy 154.94 29.21) (xy 165.1 29.21)
 		)
 		(stroke
@@
 		)
 	)
-	(label "5V_{IN}"
-		(at 166.37 29.21 180)
-		(fields_autoplaced yes)
-		(effects
-			(font
-				(size 1.27 1.27)
-			)
-			(justify right bottom)
-		)
-	)
 	(label "QSPI_SD0"
 		(at 142.24 109.22 0)
@@
 		)
 	)
+	(hierarchical_label "5V_{IN}"
+		(shape input)
+		(at 165.1 29.21 0)
+		(fields_autoplaced yes)
+		(effects
+			(font
+				(size 1.27 1.27)
+			)
+			(justify left)
+		)
+	)
 	(hierarchical_label "CRIT"
 		(shape input)
@@
 	)
 	(hierarchical_label "EN(3V)"
-		(shape input)
+		(shape output)
 		(at 106.68 93.98 0)
 		(fields_autoplaced yes)
@@
 	)
 	(hierarchical_label "EN(5V)"
-		(shape input)
+		(shape output)
 		(at 106.68 96.52 0)
 		(fields_autoplaced yes)

Commit message: Feat[SmartPowerBoard]: Routing Complete
Connections:
- net GPIO15: now reaches U6.18 (GPIO15)
- net GPIO4: no longer names the net of U6.6 (GPIO4)
Changed lines of the file:
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@@
-	)
-	(no_connect
-		(at 90.17 127)
 	)
 	(no_connect
@@
 	)
 	(no_connect
+		(at 90.17 99.06)
+	)
+	(no_connect
 		(at 90.17 106.68)
 	)
@@
 	(wire
 		(pts
-			(xy 90.17 99.06) (xy 106.68 99.06)
-		)
-		(stroke
-			(width 0)
-			(type default)
-		)
-	)
-	(wire
-		(pts
 			(xy 48.26 31.75) (xy 57.15 31.75)
 		)
@@
 		(pts
 			(xy 163.83 93.98) (xy 160.02 93.98)
+		)
+		(stroke
+			(width 0)
+			(type default)
+		)
+	)
+	(wire
+		(pts
+			(xy 90.17 127) (xy 107.95 127)
 		)
 		(stroke
@@
 		)
 	)
-	(label "GPIO4"
-		(at 106.68 99.06 180)
-		(fields_autoplaced yes)
-		(effects
-			(font
-				(size 1.27 1.27)
-			)
-			(justify right bottom)
-		)
-	)
 	(label "QSPI_SCLK"
 		(at 142.24 106.68 0)
@@
 		(fields_autoplaced yes)
 		(effects
+			(font
+				(size 1.27 1.27)
+			)
+			(justify left)
+		)
+	)
+	(hierarchical_label "GPIO15"
+		(shape input)
+		(at 107.95 127 0)
+		(fields_autoplaced yes)
+		(effects
