File: fatpower/3.3VBuck.kicad_sch (KiCad schematic)
At the start: 0 parts

Commit message: Feat[Fatpower]: Add 3.3V Buck Schematic, Vin/Vout pin of buck fixed, power connectors of navigator board/ethernet switch added
Parts:
- added C11, C12: 10uF, Capacitor_SMD:C_0603_1608Metric, symbol Device:C
- added C13, C14: 0.1uF, Capacitor_SMD:C_0402_1005Metric, symbol Device:C
- added C15, C16, C17: 22uF, Capacitor_SMD:C_0603_1608Metric, symbol Device:C
- added L2: 2.2uH, Inductor_SMD:L_Bourns_SRP7028A_7.3x6.6mm, symbol Device:L_Iron
- added R10, R8: 10k, Resistor_SMD:R_0603_1608Metric, symbol Device:R
- added R9: 33.2k, Resistor_SMD:R_0603_1608Metric, symbol Device:R
- added U1: TPS563200, Package_TO_SOT_SMD:SOT-23-6, symbol Regulator_Switching:TPS563200
Connections:
- new net: R8.1, U1.5 (EN)
- new net: C14.2, L2.1, U1.2 (SW)
- new net: R10.1, R9.2, U1.4 (VFB)
- new net: C14.1, U1.6 (VBST)
- new net GND: C11.2, C12.2, C13.2, C15.2, C16.2, C17.2, R10.2, U1.1 (GND)
- new net Vin: C11.1, C12.1, C13.1, R8.2, U1.3 (VIN)
- new net Vout: C15.1, C16.1, C17.1, L2.2, R9.1
