File: 2026_SID/untitled.kicad_sch (KiCad schematic)
At the start: 0 parts

Commit message: Feat[2026_SID]: Update SID
Changed lines of the file:
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@@
+		)
+	)
+	(hierarchical_label "PWM 13"
+		(shape input)
+		(at 226.06 118.11 0)
+		(effects
+			(font
+				(size 1.27 1.27)
+			)
+			(justify left)
+		)
+	)
+	(hierarchical_label "PWM 14"
+		(shape input)
+		(at 198.12 124.46 0)
+		(effects
+			(font
+				(size 1.27 1.27)
+			)
+			(justify left)
 		)
 	)
